File: tests/fixtures/connected_move_schematic.kicad_sch (KiCad schematic)
At the start: 2 parts

Commit message: fix: harden connectivity moves for junctions
Agent-Logs-Url: https://github.com/aldiakhou/kicad-mcp/sessions/64e436b7-8882-4c69-b659-129deb21181a

Co-authored-by: aldiakhou <46491743+aldiakhou@users.noreply.github.com>
Parts:
- added R3: 4k7, symbol Device:R
- added R4: 2k2, symbol Device:R
Changed lines of the file:
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@@
+    )
+  )
+  (symbol
+    (lib_id "Device:R")
+    (at 300 100 0)
+    (uuid "sym-r3")
+    (property "Reference" "R3"
+      (at 300 96 0)
+    )
+    (property "Value" "4k7"
+      (at 300 104 0)
+    )
+  )
+  (symbol
+    (lib_id "Device:R")
+    (at 360 100 0)
+    (uuid "sym-r4")
+    (property "Reference" "R4"
+      (at 360 96 0)
+    )
+    (property "Value" "2k2"
+      (at 360 104 0)
     )
   )
@@
     (at 240 100 0)
     (uuid "label-mid")
+  )
+  (label "JUNC"
+    (at 300 100 0)
+    (uuid "label-junc")
   )
   (wire
@@
     (uuid "wire-mid")
   )
+  (wire
+    (pts (xy 300 100) (xy 320 100))
+    (uuid "wire-junc")
+  )
+  (junction
+    (xy 300 100)
+  )
+  (wire
+    (pts (xy 360 100) (xy 380 100))
+  )
 )
